Commit message: desenvolvendo a garra e demais itens

File: my_gazebo/urdf/common_properties.xacro (robot description, xacro)
@@ -1,11 +1,7 @@
 <?xml version="1.0" ?>
-<!-- =================================================================================== -->
-<!-- |    This document was autogenerated by xacro from common_properties.xacro        | -->
-<!-- |    EDITING THIS FILE BY HAND IS NOT RECOMMENDED                                 | -->
-<!-- =================================================================================== -->
-<robot name="xacro_properties">
+<robot name="xacro_properties" xmlns:xacro="http://ros.org/wiki/xacro">
   <!-- Init colour -->
   <material name="black">
-    <color rgba="0.0 0.0 0.0 1.0"/>
+      <color rgba="0.0 0.0 0.0 1.0"/>
   </material>
   <material name="dark">
@@ -25,8 +21,8 @@
   </material>
   <material name="orange">
-    <color rgba="1.0 0.4235294117647059 0.0392156862745098 1.0"/>
+    <color rgba="${255/255} ${108/255} ${10/255} 1.0"/>
   </material>
   <material name="brown">
-    <color rgba="0.8705882352941177 0.8117647058823529 0.7647058823529411 1.0"/>
+    <color rgba="${222/255} ${207/255} ${195/255} 1.0"/>
   </material>
   <material name="red">

File: my_gazebo/urdf/turtlebot3_burger_insper.urdf (robot description, URDF)
Before this commit: robot turtlebot3_burger_insper, 10 links, 9 joints
Links:
- removed link servo_garra1_link
- added link base_camera1, mass 0.0001; collision mesh filename=package://insperbot/meshes/garra/base_camera1.stl scale=0.001 0.001 0.001; visual mesh filename=package://insperbot/meshes/garra/base_camera1.stl scale=0.001 0.001 0.001
- added link bumper_link, mass 0.0000000001; collision cylinder length=0.015 radius=0.015; visual cylinder length=0.015 radius=0.015
- added link camera_link; collision box size=0.005 0.030 0.027; visual box size=0.005 0.030 0.027
- added link camera_rgb_frame
- added link camera_rgb_optical_frame
- added link garra1garradireita1, mass 0.80e-02; collision mesh filename=package://insperbot/meshes/garra/direita.stl scale=0.001 0.001 0.001; visual mesh filename=package://insperbot/meshes/garra/direita.stl scale=0.001 0.001 0.001
- added link garra1garraesquerda1, mass 0.80e-03; collision mesh filename=package://insperbot/meshes/garra/esquerda.stl scale=0.001 0.001 0.001; visual mesh filename=package://insperbot/meshes/garra/esquerda.stl scale=0.001 0.001 0.001
- added link lat11, mass 0.0001; collision mesh filename=package://insperbot/meshes/garra/lat11.stl scale=0.001 0.001 0.001; visual mesh filename=package://insperbot/meshes/garra/lat11.stl scale=0.001 0.001 0.001
- added link lat21, mass 0.0001; collision mesh filename=package://insperbot/meshes/garra/lat21.stl scale=0.001 0.001 0.001; visual mesh filename=package://insperbot/meshes/garra/lat21.stl scale=0.001 0.001 0.001
- added link lat31, mass 0.0001; collision mesh filename=package://insperbot/meshes/garra/lat31.stl scale=0.001 0.001 0.001; visual mesh filename=package://insperbot/meshes/garra/lat31.stl scale=0.001 0.001 0.001
- added link servo_garra1, mass 0.001; collision mesh filename=package://insperbot/meshes/garra/servo_garra1.stl scale=0.001 0.001 0.001; visual mesh filename=package://insperbot/meshes/garra/servo_garra1.stl scale=0.001 0.001 0.001
Joints:
- removed joint servo_garra1_joint
- added joint Rigid1: type fixed, parent base_link_garra, child lat31, origin xyz=0.007563 -0.0205 0.001 rpy=0 0 0
- added joint Rigid2: type fixed, parent base_link_garra, child lat11, origin xyz=-0.016 0.0 0.001 rpy=0 0 0
- added joint Rigid3: type fixed, parent base_link_garra, child lat21, origin xyz=-0.002445 0.0205 0.001 rpy=0 0 0
- added joint Rigid4: type fixed, parent base_link_garra, child servo_garra1, origin xyz=0.003609 -5.8e-05 0.004 rpy=0 0 0
- added joint Rigid5: type fixed, parent lat31, child base_camera1, origin xyz=-0.002525 0.0 0.0242 rpy=0 0 0
- added joint bumper_joint: type fixed, parent base_link, child bumper_link, origin xyz=0.04 0.0 0.015 rpy=0.0 0.0 0.0
- added joint camera_joint: type fixed, parent base_link, child camera_link, origin xyz=0.05 -0.011 0.138 rpy=0 0.0 0
- added joint camera_rgb_joint: type fixed, parent camera_link, child camera_rgb_frame, origin xyz=0.003 0.011 0.009 rpy=0 0 0
- added joint camera_rgb_optical_joint: type fixed, parent camera_rgb_frame, child camera_rgb_optical_frame, origin xyz=0 0 0 rpy=-1.57 0 -1.57
- added joint joint2: type revolute, parent garra1garrabraco1, child garra1garradireita1, origin xyz=-0.0041 0.076989 0.0065 rpy=0 0 0, axis 0.0 -0.0 1.0, limit lower=-1 upper=0 effort=1 velocity=0.1
- added joint joint3: type revolute, parent garra1garrabraco1, child garra1garraesquerda1, origin xyz=-0.021 0.078672 0.0065 rpy=0 0 0, axis 0.0 -0.0 -1.0, limit lower=-1 upper=0 effort=1 velocity=0.1, mimic joint=joint2 multiplier=1 offset=0
- joint joint1: limit lower=-1.50 upper=1.5 velocity=0.1 -> lower=-1.50 upper=1.5 effort=1 velocity=0.1; origin xyz=0.083 -0.005 0.092 rpy=0 0 0 -> xyz=0.0235 0.01 0.01 rpy=0 0 0; parent servo_garra1_link -> servo_garra1; type fixed -> revolute
