Commit message: ajustes no URDF do robo - ainda sem sucesso

File: my_gazebo/urdf/turtlebot3_burger_insper.urdf (robot description, URDF)
Before this commit: robot turtlebot3_burger_insper, 7 links, 6 joints
Links:
- added link base_link_garra, mass 0.0001; collision mesh filename=package://insperbot/meshes/garra/base_link_garra.stl scale=0.001 0.001 0.001; visual mesh filename=package://insperbot/meshes/garra/base_link_garra.stl scale=0.001 0.001 0.001
- added link garra1garrabraco1, mass 2.8498940e-03; collision mesh filename=package://insperbot/meshes/garra/arm.stl scale=0.001 0.001 0.001; visual mesh filename=package://insperbot/meshes/garra/arm.stl scale=0.001 0.001 0.001
- added link servo_garra1_link, mass 0.001; collision mesh filename=package://insperbot/meshes/garra/servo_garra1.stl scale=0.001 0.001 0.001; visual mesh filename=package://insperbot/meshes/garra/servo_garra1.stl scale=0.001 0.001 0.001
- link base_link: geometry collision box size=0.140 0.140 0.143; visual mesh filename=package://insperbot/meshes/bases/burger_base.stl scale=0.001 0.001 0.001
- link base_scan: geometry collision cylinder length=0.0315 radius=0.055; visual mesh filename=package://insperbot/meshes/sensors/lds.stl scale=0.001 0.001 0.001
- link wheel_left_link: geometry collision cylinder length=0.018 radius=0.033; visual mesh filename=package://insperbot/meshes/wheels/left_tire.stl scale=0.001 0.001 0.001
- link wheel_right_link: geometry collision cylinder length=0.018 radius=0.033; visual mesh filename=package://insperbot/meshes/wheels/right_tire.stl scale=0.001 0.001 0.001
Joints:
- added joint base_joint_garra: type fixed, parent base_link, child base_link_garra, origin xyz=0.044 0.005 0.108 rpy=0 0 -1.57
- added joint joint1: type revolute, parent servo_garra1_link, child garra1garrabraco1, origin xyz=0.083 -0.005 0.092 rpy=0 0 0, axis 1.0 0.0 0.0, limit lower=-1.50 upper=1.5 effort=1 velocity=0.1
- added joint servo_garra1_joint: type fixed, parent base_link_garra, child servo_garra1_link, origin xyz=0.003609 -5.8e-05 0.004 rpy=0 0 0

Commit message: ajuste nos joints

File: my_gazebo/urdf/turtlebot3_burger_insper.urdf (robot description, URDF)
Before this commit: robot turtlebot3_burger_insper, 10 links, 9 joints
Joints:
- joint joint1: limit lower=-1.50 upper=1.5 effort=1 velocity=0.1 -> lower=-1.50 upper=1.5 velocity=0.1; type revolute -> fixed

Commit message: ajustes robo

File: my_gazebo/urdf/turtlebot3_burger_insper.urdf (robot description, URDF)
Before this commit: robot turtlebot3_burger_insper, 7 links, 6 joints
Links:
- added link garra1garrabraco1; collision mesh ; visual mesh 
- added link suportes; collision mesh ; visual mesh 
Joints:
- added joint arm_joint: type revolute, parent , child , axis 
- added joint suportes_joint: type fixed, parent , child , axis 

Commit message: mundo ok robo nao ok

File: my_gazebo/urdf/turtlebot3_burger_insper.urdf (robot description, URDF)
Before this commit: robot mybot, 20 links, 19 joints
Links:
- removed link bumper_link
- removed link camera_link
- removed link camera_rgb_frame
- removed link camera_rgb_optical_frame
- removed link garra1garradireita1
- removed link garra1garraesquerda1
- link base_camera1: mass 0.0001 -> 0.001
- link base_link: geometry collision box size=0.140 0.140 0.143; visual mesh filename=package://my_gazebo/models/turtlebot3_common/meshes/burger_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 scale=0.001 0.001 0.001
- link base_link_garra: mass 0.0001 -> 0.001
- link base_scan: geometry collision cylinder length=0.0315 radius=0.055; visual mesh filename=package://my_gazebo/models/insperbot/meshes/sensors/lds.dae scale=0.001 0.001 0.001
- link garra1garrabraco1: mass 2.8498940e-03 -> 0.00285
- link lat11: mass 0.0001 -> 0.001; geometry collision mesh filename=package://my_gazebo/models/insperbot/meshes/garra/lat11.stl scale=0.001 0.001 0.001; visual mesh filename=package://my_gazebo/models/insperbot/meshes/garra/lat11.stl scale=0.001 0.001 0.001
- link lat21: mass 0.0001 -> 0.001; geometry collision mesh filename=package://my_gazebo/models/insperbot/meshes/garra/lat21.stl scale=0.001 0.001 0.001; visual mesh filename=package://my_gazebo/models/insperbot/meshes/garra/lat21.stl scale=0.001 0.001 0.001
- link lat31: mass 0.0001 -> 0.001; geometry collision mesh filename=package://my_gazebo/models/insperbot/meshes/garra/lat31.stl scale=0.001 0.001 0.001; visual mesh filename=package://my_gazebo/models/insperbot/meshes/garra/lat31.stl scale=0.001 0.001 0.001
Joints:
- removed joint Rigid1
- removed joint Rigid2
- removed joint Rigid3
- removed joint Rigid4
- removed joint Rigid5
- removed joint base_joint_garra
- removed joint bumper_joint
- removed joint camera_joint
- removed joint camera_rgb_joint
- removed joint camera_rgb_optical_joint
- removed joint joint2
- removed joint joint3
- added joint base_camera1_joint: type fixed, parent base_link_garra, child base_camera1, origin xyz=0.083 -0.005 0.092 rpy=0 0 0
- added joint base_link_garra_joint: type fixed, parent base_link, child base_link_garra, origin xyz=0.043 0.0022 0.093 rpy=0 0 -1.57
- added joint lat11_joint: type fixed, parent base_link_garra, child lat11, origin xyz=0.083 -0.005 0.092 rpy=0 0 0
- added joint lat21_joint: type fixed, parent base_link_garra, child lat21, origin xyz=0.083 -0.005 0.092 rpy=0 0 0
- added joint lat31_joint: type fixed, parent base_link_garra, child lat31, origin xyz=0.045 0.042 0.092 rpy=0 0 0
- added joint servo_garra1_joint: type fixed, parent base_link_garra, child servo_garra1, origin xyz=0.083 -0.005 0.092 rpy=0 0 0
- joint joint1: axis 1.0 0.0 0.0 -> 1 0 0; limit lower=-1.50 upper=1.5 effort=1 velocity=0.1 -> lower=-1.57 upper=1.57 effort=10 velocity=1.0; origin xyz=0.0235 0.01 0.01 rpy=0 0 0 -> xyz=0 0 0 rpy=0 0 0
